File: LORA.kicad_sch (KiCad schematic)
At the start: 30 parts, among them J16 Conn_01x03_MountingPin, J3 Conn_Coaxial, U8 RAK3172-xx-8-SM-xI

Commit message: Update schematic components and properties across multiple files
- Changed capacitor values from "4.7u" to "4u7" and updated footprints from "C_0402_1005Metric" to "C_1206_3216Metric" in accelerometer.kicad_sch and nRF9151.kicad_sch.
- Updated part numbers for capacitors in accelerometer.kicad_sch and nRF9151.kicad_sch.
- Added a new resistor (R99) with value "100R" in hall_effect_sensor.kicad_sch.
- Removed unnecessary junctions in nRF9151.kicad_sch and adjusted wire connections.
- Added properties for MLX90637 and ZTPD2210 sensors in temp_sensors.kicad_sch.
Parts:
- TP2: now left out of the parts list
Changed lines of the file:
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@@
 		(body_style 1)
 		(exclude_from_sim no)
-		(in_bom yes)
+		(in_bom no)
 		(on_board yes)
 		(in_pos_files yes)
