File: LORA.kicad_sch (KiCad schematic)
At the start: 30 parts, among them J16 Conn_01x03_MountingPin, J3 Conn_Coaxial, U8 RAK3172-xx-8-SM-xI

Commit message: PCB updates
Update miscellaneous.kicad_sch to add new fiducial symbol and replace existing fiducial references

- Added a new fiducial symbol "BC_Miscellaneous:Fiducial" with ground
- Updated references in the schematic to point to the new fiducial symbol.

- Changed the DNP (Do Not Place) property for components U13 and U6 from 'no' to 'yes' to prevent placement on the PCB.
- Updated the footprint property for U13 to "BC_Memory:W25Q" to reflect the correct component footprint.
Parts:
- U8: now not fitted
Changed lines of the file:
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@@
 		(on_board yes)
 		(in_pos_files yes)
-		(dnp no)
+		(dnp yes)
 		(fields_autoplaced yes)
 		(property "Reference" "U8"
