File: temp_sensors.kicad_sch (KiCad schematic)
At the start: 10 parts

Commit message: Update schematic components and properties across multiple files
- Changed capacitor values from "4.7u" to "4u7" and updated footprints from "C_0402_1005Metric" to "C_1206_3216Metric" in accelerometer.kicad_sch and nRF9151.kicad_sch.
- Updated part numbers for capacitors in accelerometer.kicad_sch and nRF9151.kicad_sch.
- Added a new resistor (R99) with value "100R" in hall_effect_sensor.kicad_sch.
- Removed unnecessary junctions in nRF9151.kicad_sch and adjusted wire connections.
- Added properties for MLX90637 and ZTPD2210 sensors in temp_sensors.kicad_sch.
Parts:
- U1: value (none) -> MLX90637; PartNumber (none) -> MLX90637
- U2: value (none) -> ZTPD2210; PartNumber (none) -> ZTPD2210
Changed lines of the file:
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@@
 			)
 		)
-		(property "Value" ""
+		(property "Value" "MLX90637"
 			(at 163.83 74.93 0)
 			(show_name no)
@@
 		)
 		(property "Description" ""
+			(at 163.83 74.93 0)
+			(hide yes)
+			(show_name no)
+			(do_not_autoplace no)
+			(effects
+				(font
+					(size 1.27 1.27)
+				)
+			)
+		)
+		(property "PartNumber" "MLX90637"
 			(at 163.83 74.93 0)
 			(hide yes)
@@
 			)
 		)
-		(property "Value" ""
+		(property "Value" "ZTPD2210"
 			(at 163.83 96.52 0)
 			(show_name no)
@@
 			(at 163.83 96.52 0)
 			(hide yes)
+			(show_name no)
+			(do_not_autoplace no)
+			(effects
+				(font
+					(size 1.27 1.27)
+				)
+			)
+		)
+		(property "PartNumber" "ZTPD2210"
+			(at 163.83 96.52 0)
+			(hide yes)
