File: PowerLineSensorPCB.kicad_sch (KiCad schematic)
At the start: 2 parts

Commit message: Update schematic components and properties across multiple files
- Changed capacitor values from "4.7u" to "4u7" and updated footprints from "C_0402_1005Metric" to "C_1206_3216Metric" in accelerometer.kicad_sch and nRF9151.kicad_sch.
- Updated part numbers for capacitors in accelerometer.kicad_sch and nRF9151.kicad_sch.
- Added a new resistor (R99) with value "100R" in hall_effect_sensor.kicad_sch.
- Removed unnecessary junctions in nRF9151.kicad_sch and adjusted wire connections.
- Added properties for MLX90637 and ZTPD2210 sensors in temp_sensors.kicad_sch.
Parts:
- TP1: now left out of the parts list
Changed lines of the file:
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@@
 		(body_style 1)
 		(exclude_from_sim no)
-		(in_bom yes)
+		(in_bom no)
 		(on_board yes)
 		(in_pos_files yes)

Commit message: PCB routing.
Add netclass flags for power and signal in various schematics; update capacitor footprints and part numbers

- Introduced multiple netclass flags for "Power" and "Signal" in USB_Power, hall_effect_sensor, and nRF9151 schematics to enhance clarity and organization.
- Updated capacitor footprints from "C_1206_3216Metric" to "C_0402_1005Metric" and part numbers from "1206B475K500NT" to "CL05A475MP5NRNC" in accelerometer and nRF9151 schematics for consistency and accuracy.
- Updated submodule reference in kicad-libs to ensure compatibility with the latest library changes.
Changed lines of the file:
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@@
 			(justify left bottom)
 		)
-		(property "Netclass" "Signal"
-			(at 120.0404 66.04 0)
-			(show_name no)
-			(do_not_autoplace no)
-			(effects
-				(font
-					(size 1.27 1.27)
-				)
-				(justify right)
+		(property "Netclass" "USB"
+			(at 121.2596 66.04 0)
+			(show_name no)
+			(do_not_autoplace no)
+			(effects
+				(font
+					(size 1.27 1.27)
+				)
+				(justify left)
 			)
 		)
@@
 			)
 		)
+		(pin "A2" input
+			(at 163.83 85.09 0)
+			(effects
+				(font
+					(size 1.27 1.27)
+				)
+				(justify right)
+			)
+		)
 		(pin "A1" input
-			(at 163.83 85.09 0)
-			(effects
-				(font
-					(size 1.27 1.27)
-				)
-				(justify right)
-			)
-		)
-		(pin "A2" input
 			(at 163.83 91.44 0)
 			(effects

Commit message: pcb edits. remove old backups
Other:
- sheet RP_pico ports: added A3; removed EN_hall
