File: accelerometer.kicad_sch (KiCad schematic)
At the start: 5 parts, among them U7 LIS2HH12

Commit message: Update schematic components and properties across multiple files
- Changed capacitor values from "4.7u" to "4u7" and updated footprints from "C_0402_1005Metric" to "C_1206_3216Metric" in accelerometer.kicad_sch and nRF9151.kicad_sch.
- Updated part numbers for capacitors in accelerometer.kicad_sch and nRF9151.kicad_sch.
- Added a new resistor (R99) with value "100R" in hall_effect_sensor.kicad_sch.
- Removed unnecessary junctions in nRF9151.kicad_sch and adjusted wire connections.
- Added properties for MLX90637 and ZTPD2210 sensors in temp_sensors.kicad_sch.
Parts:
- C24: value 4.7u -> 4u7; footprint Capacitor_SMD:C_0402_1005Metric -> Capacitor_SMD:C_1206_3216Metric; PartNumber CL05B104KO5NNNC -> 1206B475K500NT
Changed lines of the file:
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@@
 			)
 		)
-		(property "Value" "4.7u"
+		(property "Value" "4u7"
 			(at 166.37 69.8499 0)
 			(show_name no)
@@
 			)
 		)
-		(property "Footprint" "Capacitor_SMD:C_0402_1005Metric"
+		(property "Footprint" "Capacitor_SMD:C_1206_3216Metric"
 			(at 163.5252 72.39 0)
 			(hide yes)
@@
 			)
 		)
-		(property "PartNumber" "CL05B104KO5NNNC"
+		(property "PartNumber" "1206B475K500NT"
 			(at 162.56 68.58 0)
 			(hide yes)

Commit message: PCB routing.
Add netclass flags for power and signal in various schematics; update capacitor footprints and part numbers

- Introduced multiple netclass flags for "Power" and "Signal" in USB_Power, hall_effect_sensor, and nRF9151 schematics to enhance clarity and organization.
- Updated capacitor footprints from "C_1206_3216Metric" to "C_0402_1005Metric" and part numbers from "1206B475K500NT" to "CL05A475MP5NRNC" in accelerometer and nRF9151 schematics for consistency and accuracy.
- Updated submodule reference in kicad-libs to ensure compatibility with the latest library changes.
Parts:
- C24: footprint Capacitor_SMD:C_1206_3216Metric -> Capacitor_SMD:C_0402_1005Metric; PartNumber 1206B475K500NT -> CL05A475MP5NRNC
Changed lines of the file:
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@@
 			)
 		)
-		(property "Footprint" "Capacitor_SMD:C_1206_3216Metric"
+		(property "Footprint" "Capacitor_SMD:C_0402_1005Metric"
 			(at 163.5252 72.39 0)
 			(hide yes)
@@
 			)
 		)
-		(property "PartNumber" "1206B475K500NT"
+		(property "PartNumber" "CL05A475MP5NRNC"
 			(at 162.56 68.58 0)
 			(hide yes)
