File: hall_effect_sensor.kicad_sch (KiCad schematic)
At the start: 15 parts, among them U11 LM2903, U5 TMAG5253BAx

Commit message: Update schematic components and properties across multiple files
- Changed capacitor values from "4.7u" to "4u7" and updated footprints from "C_0402_1005Metric" to "C_1206_3216Metric" in accelerometer.kicad_sch and nRF9151.kicad_sch.
- Updated part numbers for capacitors in accelerometer.kicad_sch and nRF9151.kicad_sch.
- Added a new resistor (R99) with value "100R" in hall_effect_sensor.kicad_sch.
- Removed unnecessary junctions in nRF9151.kicad_sch and adjusted wire connections.
- Added properties for MLX90637 and ZTPD2210 sensors in temp_sensors.kicad_sch.
Parts:
- added R99: 100R, Resistor_SMD:R_0402_1005Metric, symbol Device:R
- U5: PartNumber (none) -> TMAG5253BA1
Connections:
- net 50Hz: now also R99.1; no longer R16.1, R25.1, U11.1
- new net: R16.1, R25.1, R99.2, U11.1
Changed lines of the file:
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@@
 	(wire
 		(pts
+			(xy 52.07 118.11) (xy 55.88 118.11)
+		)
+		(stroke
+			(width 0)
+			(type default)
+		)
+	)
+	(wire
+		(pts
 			(xy 76.2 166.37) (xy 76.2 171.45)
 		)
@@
 	(wire
 		(pts
-			(xy 39.37 118.11) (xy 55.88 118.11)
+			(xy 39.37 118.11) (xy 44.45 118.11)
 		)
 		(stroke
@@
 	)
 	(symbol
+		(lib_id "Device:R")
+		(at 48.26 118.11 90)
+		(unit 1)
+		(body_style 1)
+		(exclude_from_sim no)
+		(in_bom yes)
+		(on_board yes)
+		(in_pos_files yes)
+		(dnp no)
+		(property "Reference" "R99"
+			(at 47.244 116.078 90)
+			(show_name no)
+			(do_not_autoplace no)
+			(effects
+				(font
+					(size 1.27 1.27)
+				)
+			)
+		)
+		(property "Value" "100R"
+			(at 48.26 118.11 90)
+			(show_name no)
+			(do_not_autoplace no)
+			(effects
+				(font
+					(size 1.27 1.27)
+				)
+			)
+		)
+		(property "Footprint" "Resistor_SMD:R_0402_1005Metric"
+			(at 48.26 119.888 90)
+			(hide yes)
+			(show_name no)
+			(do_not_autoplace no)
+			(effects
+				(font
+					(size 1.27 1.27)
+				)
+			)
+		)
+		(property "Datasheet" ""
+			(at 48.26 118.11 0)
+			(hide yes)
+			(show_name no)
+			(do_not_autoplace no)
+			(effects
+				(font
+					(size 1.27 1.27)
+				)
+			)
+		)
+		(property "Description" "Resistor"
+			(at 48.26 118.11 0)
+			(hide yes)
+			(show_name no)
+			(do_not_autoplace no)
+			(effects
+				(font
+					(size 1.27 1.27)
+				)
+			)
+		)
+		(property "PartNumber" "0402WGF1000TCE"
+			(at 48.26 118.11 90)
+			(hide yes)
+			(show_name no)
+			(do_not_autoplace no)
+			(effects
+				(font
+					(size 1.27 1.27)
+				)
+			)
+		)
+		(property "KLC_S4.2_DVDD" ""
+			(at 48.26 118.11 90)
+			(hide yes)
+			(show_name no)
+			(do_not_autoplace no)
+			(effects
+				(font
+					(size 1.27 1.27)
+				)
+			)
+		)
+		(property "KLC_S4.2_VREG_LX" ""
+			(at 48.26 118.11 90)
+			(hide yes)
+			(show_name no)
+			(do_not_autoplace no)
+			(effects
+				(font
+					(size 1.27 1.27)
+				)
+			)
+		)
+		(property "KLC_S3.3" ""
+			(at 48.26 118.11 90)
+			(hide yes)
+			(show_name no)
+			(do_not_autoplace no)
+			(effects
+				(font
+					(size 1.27 1.27)
+				)
+			)
+		)
+		(property "KLC_S4.1" ""
+			(at 48.26 118.11 90)
+			(hide yes)
+			(show_name no)
+			(do_not_autoplace no)
+			(effects
+				(font
+					(size 1.27 1.27)
+				)
+			)
+		)
+		(pin "1"
+		)
+		(pin "2"
+		)
+		(instances
+			(project "PowerLineSensorPCB"
+				(path "/6b3d7a89-016e-44cc-aa76-b24fbbba08cf/928b0f3b-3ed7-4d2a-bab4-19a7f307e03c"
+					(reference "R99")
+					(unit 1)
+				)
+			)
+		)
+	)
+	(symbol
 		(lib_id "power:GND")
 		(at 50.8 68.58 0)
@@
 			(at 140.97 49.53 0)
 			(hide yes)
+			(show_name no)
+			(do_not_autoplace no)
+			(effects
+				(font
+					(size 1.27 1.27)
+				)
+			)
+		)
+		(property "PartNumber" "TMAG5253BA1"
+			(at 140.97 49.53 0)
+			(hide yes)

Commit message: pcb edits. remove old backups
Parts:
- added C42: 100n, Capacitor_SMD:C_0402_1005Metric, symbol Device:C
Connections:
- net +3.3V: now also C42.1
- net GND: now also C42.2
