File: nRF9151.kicad_sch (KiCad schematic)
At the start: 84 parts, among them J1 SIM_Card_Shielded, J10 Conn_Coaxial, J14 Conn_01x06_Pin, J15 Conn_01x03_MountingPin, J7 Conn_Coaxial, SW3 SW_Push, U13 W25Q128JVE, U14 SKY65943-11, U6 nRF9151-LAXX

Commit message: PCB updates
Update miscellaneous.kicad_sch to add new fiducial symbol and replace existing fiducial references

- Added a new fiducial symbol "BC_Miscellaneous:Fiducial" with ground
- Updated references in the schematic to point to the new fiducial symbol.

- Changed the DNP (Do Not Place) property for components U13 and U6 from 'no' to 'yes' to prevent placement on the PCB.
- Updated the footprint property for U13 to "BC_Memory:W25Q" to reflect the correct component footprint.
Parts:
- U13: footprint Package_SON:WSON-8-1EP_8x6mm_P1.27mm_EP3.4x4.3mm -> BC_Memory:W25Q; now not fitted
- U6: now not fitted
Changed lines of the file:
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@@
 		(on_board yes)
 		(in_pos_files yes)
-		(dnp no)
+		(dnp yes)
 		(property "Reference" "U13"
 			(at 26.67 109.2199 0)
@@
 			)
 		)
-		(property "Footprint" "Package_SON:WSON-8-1EP_8x6mm_P1.27mm_EP3.4x4.3mm"
+		(property "Footprint" "BC_Memory:W25Q"
 			(at 38.1 87.63 0)
 			(hide yes)
@@
 		(on_board yes)
 		(in_pos_files yes)
-		(dnp no)
+		(dnp yes)
 		(fields_autoplaced yes)
 		(property "Reference" "U6"

Commit message: send to production. v0.1, making jobset for export
Parts:
- C33, C35: PartNumber CL05B104KO5NNNC -> (none)
- U13: PartNumber W25Q128JVEIM -> W25Q128JVEIM
Changed lines of the file:
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@@
 	(generator_version "10.0")
 	(paper "A4")
+	(title_block
+		(rev "${Revision}")
+	)
 	(text "Current use 400 mA\n"
 		(exclude_from_sim no)
@@
 			)
 		)
-		(property "PartNumber" "CL05B104KO5NNNC"
+		(property "PartNumber" ""
 			(at 184.15 68.58 0)
 			(hide yes)
@@
 			)
 		)
-		(property "PartNumber" "CL05B104KO5NNNC"
+		(property "PartNumber" ""
 			(at 259.08 114.3 0)
 			(hide yes)
@@
 			)
 		)
-		(property "PartNumber" "W25Q128JVEIM "
+		(property "PartNumber" "W25Q128JVEIM"
 			(at 38.1 110.49 0)
 			(hide yes)
