File: wind_sensor.kicad_sch (KiCad schematic)
At the start: 4 parts, among them J5 Conn_01x04_Pin

Commit message: send to production. v0.1, making jobset for export
Parts:
- J5: footprint Connector_PinHeader_2.54mm:PinHeader_1x04_P2.54mm_Vertical -> Connector_PinHeader_2.54mm:PinHeader_2x02_P2.54mm_Vertical
Changed lines of the file:
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@@
 	(generator_version "10.0")
 	(paper "A4")
+	(title_block
+		(rev "${Revision}")
+	)
 	(text "I2C address:\n\n2: 0x82\n3: 0x84\n4: 0x86\n5: 0x88\n6: 0x8A\n7: 0x8C\n8: 0x8E\n9: 0x90\n10: 0x92\n11: 0x94\n12: 0x96\n13: 0x98\n14: 0x9A\n15: 0x9C\n16: 0x9E\n17: 0xA0\n18: 0xA2\n19: 0xA4\n20: 0xA6\n21: 0xA8\n22: 0xAA\n23: 0xAC\n24: 0xAE\n25: 0xB0\n26: 0xB2\n27: 0xB4\n28: 0xB6\n29: 0xB8\n30: 0xBA\n31: 0xBC\n32: 0xBE"
 		(exclude_from_sim no)
@@
 			)
 		)
-		(property "Footprint" "Connector_PinHeader_2.54mm:PinHeader_1x04_P2.54mm_Vertical"
+		(property "Footprint" "Connector_PinHeader_2.54mm:PinHeader_2x02_P2.54mm_Vertical"
 			(at 135.89 86.36 0)
 			(hide yes)
