File: _restore_backup_2026-07-08T14-55-06-319/LORA.kicad_sch (KiCad schematic)
At the start: 30 parts, among them J16 Conn_01x03_MountingPin, J3 Conn_Coaxial, U8 RAK3172-xx-8-SM-xI

Commit message: PCB development!!
Update submodule and add script for selecting non-GND vias

- Updated kicad-libs submodule to the latest commit.
- Added a new script `select_all_non_gnd_vias.py` to select all vias not connected to ground nets.
- Updated references in nRF9151 schematic from "IC1" to "U14" and from "AE1" to "ANT2".
- Modified temp_sensors schematic to add a hidden power input pin and adjusted component properties.
Parts:
- U8: footprint BC_Processors:RAK3172 -> RF_Module:RAK3172
Changed lines of the file:
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@@
 			)
 		)
-		(property "Footprint" "BC_Processors:RAK3172"
+		(property "Footprint" "RF_Module:RAK3172"
 			(at 139.7 135.382 0)
 			(hide yes)
