File: _restore_backup_2026-07-08T14-55-06-319/temp_sensors.kicad_sch (KiCad schematic)
At the start: 10 parts, among them U1 MLX90637, U2 ZTPD2210

Commit message: PCB development!!
Update submodule and add script for selecting non-GND vias

- Updated kicad-libs submodule to the latest commit.
- Added a new script `select_all_non_gnd_vias.py` to select all vias not connected to ground nets.
- Updated references in nRF9151 schematic from "IC1" to "U14" and from "AE1" to "ANT2".
- Modified temp_sensors schematic to add a hidden power input pin and adjusted component properties.
Connections:
- net GND: no longer U1.6 (GND)
Changed lines of the file:
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@@
 		(pin "5"
-		)
-		(pin "6"
 		)
 		(instances
